File: output/pcbs/Cornera/right.kicad_pcb (KiCad board)
At the start: 2 copper layers, 139.8 x 121.8 mm, 63 parts

Commit message: stls
Other:
- rule pad_to_mask_clearance: 0.05 -> 0
Changed lines of the file:
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@@
 	)
 	(setup
-		(pad_to_mask_clearance 0.05)
+		(pad_to_mask_clearance 0)
 		(allow_soldermask_bridges_in_footprints no)
 		(pcbplotparams
@@
 			(outputformat 1)
 			(mirror no)
-			(drillshape 1)
+			(drillshape 0)
 			(scaleselection 1)
 			(outputdirectory "")
